Commit message: rmul_2025hero

File: src/rm_gimbal_description/urdf/rm_gimbal.urdf.xacro (robot description, xacro)
@@ -11,5 +11,5 @@
   <link name="camera_link" />
   <joint name="camera_joint" type="fixed">
-    <origin xyz="0.085 0.000 0.035" rpy="0.0  ${-pi / 60}  ${pi / 360}" />
+    <origin xyz="0.085 0.000 0.035" rpy="0.0  ${-pi / 180}  ${-pi / 360}" />
     <parent link="gimbal_link" />
     <child link="camera_link" />

Commit message: hero

File: src/rm_gimbal_description/urdf/rm_gimbal.urdf.xacro (robot description, xacro)
@@ -11,5 +11,5 @@
   <link name="camera_link" />
   <joint name="camera_joint" type="fixed">
-    <origin xyz="0.085 0.000 0.035" rpy="0.0  ${-pi / 180}  ${-pi / 360}" />
+    <origin xyz="0.085 0.000 0.035" rpy="0.0  ${pi / 24}  ${-pi / 720}" />
     <parent link="gimbal_link" />
     <child link="camera_link" />

Commit message: final

File: src/rm_gimbal_description/urdf/rm_gimbal.urdf.xacro (robot description, xacro)
@@ -11,5 +11,5 @@
   <link name="camera_link" />
   <joint name="camera_joint" type="fixed">
-    <origin xyz="0.085 0.000 0.035" rpy="0.0  ${pi / 24}  ${-pi / 720}" />
+    <origin xyz="0.085 0.000 0.035" rpy="0.0  ${pi / 25}  ${-pi / 720}" />
     <parent link="gimbal_link" />
     <child link="camera_link" />
